File: kicad/Linky_TEMPO.kicad_pcb (KiCad board)
At the start: 2 copper layers, 62.7 x 87.8 mm, 36 parts, among them J1_EAU1 Screw_Terminal_01x03, J2_CHAUF1 Screw_Terminal_01x03, J3 Screw_Terminal_01x03, J4 Screw_Terminal_01x03, K1 SANYOU_SRD_Form_C, K2 SANYOU_SRD_Form_C, Q1 TRANS_NPN-MMBT2222AL, Q2 TRANS_NPN-MMBT2222AL, Q3 BS170F, SW1 SW_DIP_x05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

Commit message: Update pcb Kicad 1.0.1
Update pcb Kicad 1.0.1
Parts:
- moved G*** 2.83 mm to (170.6, 94.8)
Routing:
- added copper zone on F.Cu, net GND
Other:
- outline, holes or cut-outs redrawn
- board text added: "FuméeBleue - V1.01"
- board text removed: "FuméeBleue - V1.00"
Changed lines of the file:
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@@
   )
   (paper "A4")
+  (title_block
+    (comment 4 "AISLER Project ID: KVRGMSSR")
+  )
   (layers
     (0 "F.Cu" signal)
@@
   )
   (footprint "logo_fb:logo_fb_small" (layer "F.Cu")
-    (at 167.8 95.2 90)
+    (at 170.6 94.8 90)
     (attr board_only exclude_from_pos_files exclude_from_bom)
     (fp_text reference "G***" (at 0 0 90) (layer "F.SilkS") hide
@@
   (gr_arc (start 112.52132 59.19632) (mid 113.4 57.075) (end 115.52132 56.19632) (layer "Edge.Cuts") (width 0.1))
   (gr_line (start 175.250183 144) (end 175.235953 59.214386) (layer "Edge.Cuts") (width 0.1))
-  (gr_circle (center 171.5 102.25) (end 173 103.75) (layer "Edge.Cuts") (width 0.1) (fill none))
+  (gr_circle (center 171.5 103) (end 173.62132 103) (layer "Edge.Cuts") (width 0.1) (fill none))
   (gr_line (start 172.235953 56.214386) (end 115.52132 56.19632) (layer "Edge.Cuts") (width 0.1))
   (gr_arc (start 172.235953 56.214386) (mid 174.357273 57.093066) (end 175.235953 59.214386) (layer "Edge.Cuts") (width 0.1))
   (gr_circle (center 116 103) (end 117.5 104.5) (layer "Edge.Cuts") (width 0.1) (fill none))
-  (gr_text "FuméeBleue - V1.00" (at 173.2 82.4 270) (layer "F.SilkS")
+  (gr_text "FuméeBleue - V1.01" (at 173.2 78.6 270) (layer "F.SilkS")
     (effects (font (size 1.5 1.5) (thickness 0.3)))
   )
@@
   (segment (start 165.235 85.1075) (end 165.235 86.415) (width 0.3) (layer "F.Cu") (net 52))
   (segment (start 158 89.575) (end 161.55 89.575) (width 0.3) (layer "F.Cu") (net 52))
+  (zone (net 4) (net_name "GND") (layer "F.Cu") (hatch edge 0.508)
+    (connect_pads (clearance 0.508))
+    (min_thickness 0.254) (filled_areas_thickness no)
+    (fill yes (thermal_gap 0.508) (thermal_bridge_width 0.508))
+    (polygon
+      (pts
+        (xy 176.2 109.2)
+        (xy 112 109)
+        (xy 112 55.6)
+        (xy 176.2 55.6)
+      )
+    )
+  )
   (zone (net 4) (net_name "GND") (layer "B.Cu") (hatch edge 0.508)
     (connect_pads (clearance 0.508))

Commit message: v1.0.1 PCB
v1.0.1 PCB Kicad
Parts:
- removed the REF** at (116.0, 110.6)
- removed the REF** at (143.2, 120.8)
- added REF**: WEEE-Logo_8.4x12mm_SilkScreen, Symbol:WEEE-Logo_8.4x12mm_SilkScreen, F.Cu at (122.6, 106.2)
- R10, R9: value 1k -> 10k
- R11, R3, R4, R5, R6, R7: value 1k -> 1,2k
Connections:
- A1 pad 11: unconnected-(A1-Pad11) -> Net-(D5-Pad2)
- A1 pad 12: unconnected-(A1-Pad12) -> Net-(D4-Pad2)
- A1 pad 13: unconnected-(A1-Pad13) -> Net-(D3-Pad2)
- A1 pad 24: Net-(A1-Pad24) -> unconnected-(A1-Pad24)
- A1 pad 25: Net-(A1-Pad25) -> unconnected-(A1-Pad25)
- A1 pad 26: Net-(A1-Pad26) -> unconnected-(A1-Pad26)
- D3 pad 2: Net-(A1-Pad24) -> Net-(D3-Pad2)
- D4 pad 2: Net-(A1-Pad25) -> Net-(D4-Pad2)
- D5 pad 2: Net-(A1-Pad26) -> Net-(D5-Pad2)
Routing:
- net Net-(D5-Pad2): track 0.00 -> 49.5 mm
- net Net-(D4-Pad2): track 0.00 -> 45.5 mm
- net Net-(D3-Pad2): track 0.00 -> 44.7 mm
- net Net-(A1-Pad26): track 24.4 -> 0.00 mm
- net Net-(A1-Pad24): track 24.0 -> 0.00 mm
- net Net-(A1-Pad25): track 23.6 -> 0.00 mm

Commit message: PCB v1.01
Parts:
- removed REF**: WEEE-Logo_8.4x12mm_SilkScreen, Symbol:WEEE-Logo_8.4x12mm_SilkScreen
- R1: value 1,2k -> 1k
- R11, R3, R4, R5, R6: value 1,2k -> 2,2k
- R2: value 10k -> 3.3k
- R7: value 1,2k -> 2,2
