File: kicad/Linky_TEMPO.kicad_sch (KiCad schematic)
At the start: 33 parts, among them J1_EAU1 Screw_Terminal_01x03, J2_CHAUF1 Screw_Terminal_01x03, J3 Screw_Terminal_01x03, J4 Screw_Terminal_01x03, K1 SANYOU_SRD_Form_C, K2 SANYOU_SRD_Form_C, Q1 TRANS_NPN-MMBT2222AL, Q2 TRANS_NPN-MMBT2222AL, Q3 BS170F, SW1 SW_DIP_x05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

Commit message: Update pcb Kicad 1.0.1
Update pcb Kicad 1.0.1
Parts:
- R10, R9: value 1k -> 10k
- R11, R3, R4, R5, R6, R7: value 1k -> 470
Changed lines of the file:
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@@
   (title_block
     (title "Linky_TEMPO")
+    (rev "v1.01")
     (company "FuméeBleue")
   )
@@
     (in_bom yes) (on_board yes) (fields_autoplaced)
     (property "Reference" "R9" (id 0) (at 149.86 106.68 90))
-    (property "Value" "1k" (id 1) (at 149.86 109.22 90))
+    (property "Value" "10k" (id 1) (at 149.86 109.22 90))
     (property "Footprint" "Resistor_SMD:R_1206_3216Metric" (id 2) (at 149.86 111.252 90))
     (property "Datasheet" "~" (id 3) (at 149.86 113.03 0)
@@
   (symbol (lib_id "Device:R") (at 196.85 119.38 270) (unit 1)
     (in_bom yes) (on_board yes)
-    (property "Reference" "R6" (id 0) (at 196.85 113.03 90))
-    (property "Value" "1k" (id 1) (at 196.85 115.57 90))
+    (property "Reference" "R6" (id 0) (at 196.85 120.65 90))
+    (property "Value" "470" (id 1) (at 196.85 119.38 90))
     (property "Footprint" "Resistor_SMD:R_1206_3216Metric" (id 2) (at 196.85 117.602 90)
       (effects (font (size 1.27 1.27)) hide)
@@
   (symbol (lib_id "Device:R") (at 196.85 115.57 270) (unit 1)
     (in_bom yes) (on_board yes)
-    (property "Reference" "R5" (id 0) (at 200.66 109.22 90))
-    (property "Value" "1k" (id 1) (at 200.66 111.76 90))
+    (property "Reference" "R5" (id 0) (at 196.85 116.84 90))
+    (property "Value" "470" (id 1) (at 196.85 115.57 90))
     (property "Footprint" "Resistor_SMD:R_1206_3216Metric" (id 2) (at 196.85 113.792 90)
       (effects (font (size 1.27 1.27)) hide)
@@
     (in_bom yes) (on_board yes) (fields_autoplaced)
     (property "Reference" "R10" (id 0) (at 149.86 109.22 90))
-    (property "Value" "1k" (id 1) (at 149.86 111.76 90))
+    (property "Value" "10k" (id 1) (at 149.86 111.76 90))
     (property "Footprint" "Resistor_SMD:R_1206_3216Metric" (id 2) (at 149.86 113.792 90)
       (effects (font (size 1.27 1.27)) hide)
@@
   )
   (symbol (lib_id "Device:R") (at 196.85 123.19 270) (unit 1)
-    (in_bom yes) (on_board yes) (fields_autoplaced)
-    (property "Reference" "R7" (id 0) (at 196.85 116.84 90))
-    (property "Value" "1k" (id 1) (at 196.85 119.38 90))
+    (in_bom yes) (on_board yes)
+    (property "Reference" "R7" (id 0) (at 196.85 124.46 90))
+    (property "Value" "470" (id 1) (at 196.85 123.19 90))
     (property "Footprint" "Resistor_SMD:R_1206_3216Metric" (id 2) (at 196.85 121.412 90)
       (effects (font (size 1.27 1.27)) hide)
@@
   (symbol (lib_id "Device:R") (at 142.24 100.33 270) (unit 1)
     (in_bom yes) (on_board yes)
-    (property "Reference" "R11" (id 0) (at 142.24 93.98 90))
-    (property "Value" "1k" (id 1) (at 142.24 96.52 90))
+    (property "Reference" "R11" (id 0) (at 142.24 102.87 90))
+    (property "Value" "470" (id 1) (at 142.24 100.33 90))
     (property "Footprint" "Resistor_SMD:R_1206_3216Metric" (id 2) (at 142.24 98.552 90)
       (effects (font (size 1.27 1.27)) hide)
@@
   )
   (symbol (lib_id "Device:R") (at 142.24 87.63 270) (unit 1)
-    (in_bom yes) (on_board yes) (fields_autoplaced)
-    (property "Reference" "R3" (id 0) (at 142.24 81.28 90))
-    (property "Value" "1k" (id 1) (at 142.24 83.82 90))
+    (in_bom yes) (on_board yes)
+    (property "Reference" "R3" (id 0) (at 142.24 85.09 90))
+    (property "Value" "470" (id 1) (at 142.24 87.63 90))
     (property "Footprint" "Resistor_SMD:R_1206_3216Metric" (id 2) (at 142.24 85.852 90)
       (effects (font (size 1.27 1.27)) hide)
@@
   )
   (symbol (lib_id "Device:R") (at 142.24 90.17 270) (unit 1)
-    (in_bom yes) (on_board yes) (fields_autoplaced)
-    (property "Reference" "R4" (id 0) (at 142.24 83.82 90))
-    (property "Value" "1k" (id 1) (at 142.24 86.36 90))
+    (in_bom yes) (on_board yes)
+    (property "Reference" "R4" (id 0) (at 142.24 92.71 90))
+    (property "Value" "470" (id 1) (at 142.24 90.17 90))
     (property "Footprint" "Resistor_SMD:R_1206_3216Metric" (id 2) (at 142.24 88.392 90)
       (effects (font (size 1.27 1.27)) hide)
@@
     )
     (path "/adb0036a-8d7f-4d84-8fa0-c0e5f1b6072f"
-      (reference "R3") (unit 1) (value "1k") (footprint "Resistor_SMD:R_1206_3216Metric")
+      (reference "R3") (unit 1) (value "470") (footprint "Resistor_SMD:R_1206_3216Metric")
     )
     (path "/ce0c7769-8b5d-4cbb-a785-5a0fc5f2e795"
-      (reference "R4") (unit 1) (value "1k") (footprint "Resistor_SMD:R_1206_3216Metric")
+      (reference "R4") (unit 1) (value "470") (footprint "Resistor_SMD:R_1206_3216Metric")
     )
     (path "/339a66d9-aa64-45e0-b084-36d8731fed88"
-      (reference "R5") (unit 1) (value "1k") (footprint "Resistor_SMD:R_1206_3216Metric")
+      (reference "R5") (unit 1) (value "470") (footprint "Resistor_SMD:R_1206_3216Metric")
     )
     (path "/32b1d3c8-868a-409b-921f-3fd3e674d422"
-      (reference "R6") (unit 1) (value "1k") (footprint "Resistor_SMD:R_1206_3216Metric")
+      (reference "R6") (unit 1) (value "470") (footprint "Resistor_SMD:R_1206_3216Metric")
     )
     (path "/8128c63b-004d-4030-b5d5-fe6802715502"
-      (reference "R7") (unit 1) (value "1k") (footprint "Resistor_SMD:R_1206_3216Metric")
+      (reference "R7") (unit 1) (value "470") (footprint "Resistor_SMD:R_1206_3216Metric")
     )
     (path "/9eeb528d-5112-4c2c-9657-2b787b811a11"
@@
     )
     (path "/1195f711-2c5b-412c-8467-4a1fefa4dd5e"
-      (reference "R9") (unit 1) (value "1k") (footprint "Resistor_SMD:R_1206_3216Metric")
+      (reference "R9") (unit 1) (value "10k") (footprint "Resistor_SMD:R_1206_3216Metric")
     )
     (path "/57f4a0ea-e9c1-4f73-b7bd-95f59e744ead"
-      (reference "R10") (unit 1) (value "1k") (footprint "Resistor_SMD:R_1206_3216Metric")
+      (reference "R10") (unit 1) (value "10k") (footprint "Resistor_SMD:R_1206_3216Metric")
     )
     (path "/87dcddab-dc7f-43d2-945d-99d3f67c0479"
-      (reference "R11") (unit 1) (value "1k") (footprint "Resistor_SMD:R_1206_3216Metric")
+      (reference "R11") (unit 1) (value "470") (footprint "Resistor_SMD:R_1206_3216Metric")
     )
     (path "/a053ea8d-528d-4e4e-a6a6-9c10b81fd410"

Commit message: v1.0.1 PCB
v1.0.1 PCB Kicad
Parts:
- R11, R3, R4, R5, R6, R7: value 470 -> 1,2k
Connections:
- net at A1.11 (D8): now also D5.2 (A)
- net at A1.12 (D9): now also D4.2 (A)
- net at A1.13 (D10): now also D3.2 (A)
- net at A1.24 (A5): no longer D3.2 (A)
- net at A1.25 (A6): no longer D4.2 (A)
- net at A1.26 (A7): no longer D5.2 (A)
- no-connect marks 10 -> 7
Other:
- moved on the sheet: D3, D4, D5, R5, R6, R7

Commit message: PCB v1.01
Parts:
- R1: value 1,2k -> 1k
- R11, R3, R4, R5, R6: value 1,2k -> 2,2k
- R2: value 10k -> 3.3k
- R7: value 1,2k -> 2,2
Connections:
- no-connect marks 7 -> 10
